File: Fula52/Fula52.kicad_pcb (KiCad board)
At the start: 2 copper layers, 231.1 x 97.8 mm, 149 parts, among them J1 USB_C_Receptacle_USB2.0, SW1 BOOT, SW2 RESET, U1 RT9013-33GB, U2 SRV05-4, U3 W25Q128JVS, U4 RP2040, Y1 12MHz

Commit message: full routed
Parts:
- removed TP1, TP4: TestPoint, TestPoint:TestPoint_Pad_D2.5mm
- added SB1: SolderJumper_2_Open, Jumper:SolderJumper-2_P1.3mm_Open_TrianglePad1.0x1.5mm, B.Cu at (35.8, 53.0)
- moved R3 2.39 mm to (34.3, 51.4), turned to -135 degrees
- moved C12 0.97 mm to (45.8, 70.6)
- moved LD1 0.67 mm to (33.0, 50.2), turned to -135 degrees
- moved U3 0.66 mm to (63.5, 65.5)
- moved C3 0.66 mm to (59.8, 62.0)
- moved R6 0.66 mm to (67.0, 62.0)
- moved R7 0.66 mm to (65.0, 62.0)
- moved SW1 0.20 mm to (71.8, 54.7)
- moved SW2 0.20 mm to (71.8, 50.3)
Connections:
- R3 pad 2: GND -> Net-(R3-Pad2)
- U4 pad 11: COL_6 -> COL_1
- U4 pad 12: unconnected-(U4-Pad12) -> COL_6
- U4 pad 16: unconnected-(U4-Pad16) -> COL_2
- U4 pad 2: COL_11 -> unconnected-(U4-Pad2)
- U4 pad 28: COL_2 -> unconnected-(U4-Pad28)
- U4 pad 3: COL_10 -> unconnected-(U4-Pad3)
- U4 pad 30: COL_1 -> ROW_1
- U4 pad 31: unconnected-(U4-Pad31) -> ROW_2
- U4 pad 32: ROW_4 -> unconnected-(U4-Pad32)
- U4 pad 34: ROW_3 -> unconnected-(U4-Pad34)
- U4 pad 35: ROW_2 -> unconnected-(U4-Pad35)
- U4 pad 36: unconnected-(U4-Pad36) -> ROW_3
- U4 pad 37: ROW_1 -> ROW_4
- U4 pad 38: unconnected-(U4-Pad38) -> COL_0
- U4 pad 39: COL_0 -> STATE_LED
- U4 pad 4: unconnected-(U4-Pad4) -> COL_11
- U4 pad 41: STATE_LED -> unconnected-(U4-Pad41)
- U4 pad 5: COL_9 -> COL_10
- U4 pad 6: unconnected-(U4-Pad6) -> COL_9
Routing:
- net COL_11: track 64.4 -> 265.1 mm
- net COL_10: track 64.4 -> 245.8 mm
- net COL_9: track 64.4 -> 226.6 mm
- net ROW_4: track 71.4 -> 217.7 mm
- net COL_8: track 64.4 -> 207.4 mm
- net COL_7: track 88.5 -> 212.3 mm
- net COL_6: track 86.5 -> 193.3 mm
- net COL_5: track 84.6 -> 172.1 mm
- net COL_4: track 86.4 -> 154.8 mm
- net /RP2040/~{RESET}: track 6.85 -> 71.2 mm, vias 2 -> 4
- net ROW_3: track 209.6 -> 271.3 mm
- net COL_3: track 64.4 -> 110.8 mm
- net ROW_2: track 209.6 -> 249.9 mm
- net STATE_LED: track 0.00 -> 28.4 mm
- net COL_2: track 64.4 -> 91.8 mm
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Other:
- outline, holes or cut-outs redrawn
