File: Calcite52/Calcite52.kicad_pcb (KiCad board)
At the start: 2 copper layers, 231.1 x 97.8 mm, 148 parts, among them J1 USB_C_Receptacle_USB2.0, SW1 BOOT, SW2 RESET, U1 RT9013-33GB, U2 SRV05-4, U3 W25Q128JVS, U4 RP2040, Y1 12MHz

Commit message: Update layout
Parts:
- added G***: LOGO, LOGO, B.Cu at (218.5, 135.5)
- added G***: LOGO, LOGO, B.Cu at (243.7, 132.9)

Commit message: Update layout and logo
Parts:
- added kibuzzard-63E64B4D: G***, kibuzzard-63E64B4D, B.Cu at (235.3, 134.0)
- LD1: value Red -> Blue
- moved G*** 2.40 mm to (245.4, 131.2)
- moved H6 1.77 mm to (145.4, 124.6)
- moved G*** 1.04 mm to (219.0, 134.6)
- moved R3 0.23 mm to (34.1, 51.3)
- turned SB1 to -45 degrees
Connections:
- SB1 pad 1: GND -> Net-(R3-Pad2)
- SB1 pad 2: Net-(R3-Pad2) -> GND
Routing:
- net GND: track 40.0 -> 38.6 mm, vias 42 -> 41
- net +1V1: track 23.4 -> 24.2 mm

Commit message: Update BOM
Parts:
- added H10: MountingHole, MountingHole:MountingHole_2.2mm_M2, F.Cu at (256.8, 105.5)
- added H7: MountingHole, MountingHole:MountingHole_2.2mm_M2, F.Cu at (34.0, 67.4)
- added H8: MountingHole, MountingHole:MountingHole_2.2mm_M2, F.Cu at (34.0, 105.5)
- added H9: MountingHole, MountingHole:MountingHole_2.2mm_M2, F.Cu at (256.8, 67.4)
- moved H2 19.1 mm to (202.6, 67.4)
- moved H4 19.1 mm to (202.6, 105.5)
- moved H3 19.1 mm to (88.3, 105.5)
- moved G*** 0.36 mm to (219.3, 134.5)
- moved H1 0.13 mm to (145.4, 86.5)
- moved H5 0.13 mm to (88.3, 67.4)
Routing:
- net GND: vias 41 -> 45
Other:
- board text added: "JLCJLCJLCJLC"
