File: Calcite52/Calcite52.kicad_pcb (KiCad board)
At the start: 2 copper layers, 231.1 x 97.8 mm, 155 parts, among them J1 USB_C_Receptacle_USB2.0, SW1 BOOT, SW2 RESET, U1 RT9013-33GB, U2 SRV05-4, U3 W25Q128JVS, U4 RP2040, Y1 12MHz

Commit message: Add PCB center mark at "User.4" layer
Other:
- board text added: "Center"
Changed lines of the file:
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@@
   (gr_line (start 258.445 144.78) (end 32.385 144.78) (layer "Edge.Cuts") (width 0.1))
   (gr_arc (start 260.985 142.24) (mid 260.241051 144.036051) (end 258.445 144.78) (layer "Edge.Cuts") (width 0.1))
+  (gr_circle locked (center 145.415 95.885) (end 146.415 95.885) (layer "User.4") (width 0.25) (fill none))
   (gr_text "JLCJLCJLCJLC" (at 254.381 49.3) (layer "B.SilkS")
     (effects (font (size 1 1) (thickness 0.15)) (justify mirror))
   )
+  (gr_text "Center" (at 145.415 97.79) (layer "User.4")
+    (effects (font (size 1 1) (thickness 0.15)))
+  )
   (dimension (type aligned) (layer "Dwgs.User")
