File: Calcite52/Calcite52.kicad_sch (KiCad schematic)
At the start: 19 parts, among them J1 USB_C_Receptacle_USB2.0, U1 RT9013-33GB, U2 SRV05-4

Commit message: Update layout
Other:
- note added: "ESD"
- note added: "Power"
- note added: "State LED"
- note added: "USB"
- moved on the sheet: C1, C2, LD1, R3, SB1, U1, U2

Commit message: Update layout and logo
Parts:
- LD1: value Red -> Blue; LCSC C2286 -> C72043; MFR. Part # KT-0603R -> 19-217/GHC-YR1S2/3T
Connections:
- net GND: now also SB1.2 (B); no longer SB1.1 (A)
- net at R3.2: now also SB1.1 (A); no longer SB1.2 (B)
Other:
- moved on the sheet: SB1
Changed lines of the file:
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@@
     )
   )
-  (symbol (lib_id "Jumper:SolderJumper_2_Open") (at 232.41 130.81 90) (unit 1)
+  (symbol (lib_id "Jumper:SolderJumper_2_Open") (at 232.41 130.81 270) (unit 1)
     (in_bom yes) (on_board yes) (fields_autoplaced)
     (property "Reference" "SB1" (id 0) (at 234.95 129.5399 90)
-      (effects (font (size 1.27 1.27)) (justify right))
+      (effects (font (size 1.27 1.27)) (justify left))
     )
     (property "Value" "SolderJumper_2_Open" (id 1) (at 234.95 132.0799 90)
-      (effects (font (size 1.27 1.27)) (justify right))
+      (effects (font (size 1.27 1.27)) (justify left))
     )
     (property "Footprint" "Jumper:SolderJumper-2_P1.3mm_Open_TrianglePad1.0x1.5mm" (id 2) (at 232.41 130.81 0)
@@
       (effects (font (size 1.27 1.27)) (justify right))
     )
-    (property "Value" "Red" (id 1) (at 236.22 115.8874 90)
+    (property "Value" "Blue" (id 1) (at 236.22 115.8874 90)
       (effects (font (size 1.27 1.27)) (justify right))
     )
@@
       (effects (font (size 1.27 1.27)) hide)
     )
-    (property "LCSC" "C2286" (id 4) (at 232.41 113.03 0)
-      (effects (font (size 1.27 1.27)) hide)
-    )
-    (property "MFR. Part #" "KT-0603R" (id 5) (at 232.41 113.03 0)
+    (property "LCSC" "C72043" (id 4) (at 232.41 113.03 0)
+      (effects (font (size 1.27 1.27)) hide)
+    )
+    (property "MFR. Part #" "19-217/GHC-YR1S2/3T" (id 5) (at 232.41 113.03 0)
       (effects (font (size 1.27 1.27)) hide)
     )
@@
     )
     (path "/67c6b337-141b-4cd3-b65c-03837c26cb88"
-      (reference "LD1") (unit 1) (value "Red") (footprint "LED_SMD:LED_0603_1608Metric")
+      (reference "LD1") (unit 1) (value "Blue") (footprint "LED_SMD:LED_0603_1608Metric")
     )
     (path "/ec56ede5-b45e-4b38-b253-e90af267d8d0"

Commit message: Update BOM
Parts:
- added H10, H7, H8, H9: MountingHole, MountingHole:MountingHole_2.2mm_M2, symbol Mechanical:MountingHole
Other:
- note added: "ESD Protection"
- note removed: "ESD"
Changed lines of the file:
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@@
     (stroke (width 0) (type default) (color 0 0 0 0))
   )
-  (text "ESD" (at 135.89 31.75 0)
+  (text "ESD Protection" (at 130.81 31.75 0)
     (effects (font (size 1.5 1.5) (thickness 0.3) bold) (justify left bottom))
   )
@@
     )
   )
+  (symbol (lib_id "Mechanical:MountingHole") (at 116.84 194.31 0) (unit 1)
+    (in_bom no) (on_board yes) (fields_autoplaced)
+    (property "Reference" "H7" (id 0) (at 119.38 193.0399 0)
+      (effects (font (size 1.27 1.27)) (justify left) hide)
+    )
+    (property "Value" "MountingHole" (id 1) (at 119.38 195.5799 0)
+      (effects (font (size 1.27 1.27)) (justify left) hide)
+    )
+    (property "Footprint" "MountingHole:MountingHole_2.2mm_M2" (id 2) (at 116.84 194.31 0)
+      (effects (font (size 1.27 1.27)) hide)
+    )
+    (property "Datasheet" "~" (id 3) (at 116.84 194.31 0)
+      (effects (font (size 1.27 1.27)) hide)
+    )
+  )
   (symbol (lib_id "Mechanical:MountingHole") (at 173.99 194.31 0) (unit 1)
     (in_bom no) (on_board yes) (fields_autoplaced)
@@
     (pin "1")
     (pin "2")
+  )
+  (symbol (lib_id "Mechanical:MountingHole") (at 123.19 194.31 0) (unit 1)
+    (in_bom no) (on_board yes) (fields_autoplaced)
+    (property "Reference" "H8" (id 0) (at 125.73 193.0399 0)
+      (effects (font (size 1.27 1.27)) (justify left) hide)
+    )
+    (property "Value" "MountingHole" (id 1) (at 125.73 195.5799 0)
+      (effects (font (size 1.27 1.27)) (justify left) hide)
+    )
+    (property "Footprint" "MountingHole:MountingHole_2.2mm_M2" (id 2) (at 123.19 194.31 0)
+      (effects (font (size 1.27 1.27)) hide)
+    )
+    (property "Datasheet" "~" (id 3) (at 123.19 194.31 0)
+      (effects (font (size 1.27 1.27)) hide)
+    )
   )
   (symbol (lib_id "Device:LED") (at 232.41 113.03 90) (unit 1)
@@
     (pin "2")
   )
+  (symbol (lib_id "Mechanical:MountingHole") (at 129.54 194.31 0) (unit 1)
+    (in_bom no) (on_board yes) (fields_autoplaced)
+    (property "Reference" "H9" (id 0) (at 132.08 193.0399 0)
+      (effects (font (size 1.27 1.27)) (justify left) hide)
+    )
+    (property "Value" "MountingHole" (id 1) (at 132.08 195.5799 0)
+      (effects (font (size 1.27 1.27)) (justify left) hide)
+    )
+    (property "Footprint" "MountingHole:MountingHole_2.2mm_M2" (id 2) (at 129.54 194.31 0)
+      (effects (font (size 1.27 1.27)) hide)
+    )
+    (property "Datasheet" "~" (id 3) (at 129.54 194.31 0)
+      (effects (font (size 1.27 1.27)) hide)
+    )
+  )
   (symbol (lib_id "power:GND") (at 233.68 59.69 0) (unit 1)
     (in_bom yes) (on_board yes)
@@
     )
     (pin "1")
+  )
+  (symbol (lib_id "Mechanical:MountingHole") (at 135.89 194.31 0) (unit 1)
+    (in_bom no) (on_board yes) (fields_autoplaced)
+    (property "Reference" "H10" (id 0) (at 138.43 193.0399 0)
+      (effects (font (size 1.27 1.27)) (justify left) hide)
+    )
+    (property "Value" "MountingHole" (id 1) (at 138.43 195.5799 0)
+      (effects (font (size 1.27 1.27)) (justify left) hide)
+    )
+    (property "Footprint" "MountingHole:MountingHole_2.2mm_M2" (id 2) (at 135.89 194.31 0)
+      (effects (font (size 1.27 1.27)) hide)
+    )
+    (property "Datasheet" "~" (id 3) (at 135.89 194.31 0)
+      (effects (font (size 1.27 1.27)) hide)
+    )
   )
   (symbol (lib_id "Connector:TestPoint") (at 69.85 57.15 270) (unit 1)
@@
       (reference "H6") (unit 1) (value "MountingHole") (footprint "MountingHole:MountingHole_2.2mm_M2")
     )
+    (path "/0bea03be-8935-4a18-ad68-0ec243a35635"
+      (reference "H7") (unit 1) (value "MountingHole") (footprint "MountingHole:MountingHole_2.2mm_M2")
+    )
+    (path "/61e27586-e1ea-4139-a05d-3bcf7fdfbf8b"
+      (reference "H8") (unit 1) (value "MountingHole") (footprint "MountingHole:MountingHole_2.2mm_M2")
+    )
+    (path "/69ed8bbc-0a2d-43e9-b311-cb66eecb38c2"
+      (reference "H9") (unit 1) (value "MountingHole") (footprint "MountingHole:MountingHole_2.2mm_M2")
+    )
+    (path "/83b52234-6767-45bd-af46-26940ed67f0c"
+      (reference "H10") (unit 1) (value "MountingHole") (footprint "MountingHole:MountingHole_2.2mm_M2")
+    )
     (path "/965698a2-154b-45fe-8bd1-84f3c4280877"
