File: Calcite52/RP2040.kicad_sch (KiCad schematic)
At the start: 25 parts, among them SW1 BOOT, SW2 RESET, U3 W25Q128JVS, U4 RP2040, Y1 12MHz

Commit message: Update layout
Connections:
- no-connect marks 2 -> 14
Changed lines of the file:
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@@
   (junction (at 36.83 91.44) (diameter 0) (color 0 0 0 0)
   )
+  (no_connect (at 116.84 40.64))
+  (no_connect (at 116.84 43.18))
+  (no_connect (at 116.84 83.82))
+  (no_connect (at 116.84 86.36))
+  (no_connect (at 116.84 93.98))
+  (no_connect (at 116.84 116.84))
+  (no_connect (at 116.84 58.42))
+  (no_connect (at 116.84 76.2))
+  (no_connect (at 116.84 78.74))
+  (no_connect (at 116.84 81.28))
+  (no_connect (at 116.84 96.52))
+  (no_connect (at 116.84 99.06))
   (no_connect (at 66.04 106.68))
   (no_connect (at 66.04 109.22))
@@
     (stroke (width 0) (type default) (color 0 0 0 0))
   )
-  (text "Flash" (at 222.25 34.29 0)
-    (effects (font (size 2 2) bold) (justify left bottom))
+  (text "Flash" (at 224.79 35.56 0)
+    (effects (font (size 1.5 1.5) bold) (justify left bottom))
   )
   (label "QSPI_SS" (at 54.61 58.42 0)

Commit message: Update BOM
Parts:
- SW1, SW2: LCSC (none) -> C5117871; MFR. Part # (none) -> GT-TC060B-H027-L1
Changed lines of the file:
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@@
       (effects (font (size 1.27 1.27)) hide)
     )
-    (property "MFR. Part #" "" (id 4) (at 245.11 130.81 90)
+    (property "MFR. Part #" "GT-TC060B-H027-L1" (id 4) (at 245.11 130.81 90)
       (effects (font (size 1.27 1.27)) hide)
     )
-    (property "LCSC" "" (id 6) (at 245.11 130.81 0)
+    (property "LCSC" "C5117871" (id 6) (at 245.11 130.81 0)
       (effects (font (size 1.27 1.27)) hide)
     )
@@
       (effects (font (size 1.27 1.27)) hide)
     )
-    (property "MFR. Part #" "" (id 4) (at 214.63 130.81 90)
+    (property "MFR. Part #" "GT-TC060B-H027-L1" (id 4) (at 214.63 130.81 90)
       (effects (font (size 1.27 1.27)) hide)
     )
-    (property "LCSC" "" (id 6) (at 214.63 130.81 0)
+    (property "LCSC" "C5117871" (id 6) (at 214.63 130.81 0)
       (effects (font (size 1.27 1.27)) hide)
     )
