File: Calcite60/pcb/RP2040.kicad_sch (KiCad schematic)
At the start: 25 parts, among them SW1 BOOT, SW2 RESET, U3 W25Q128JVS, U4 RP2040, Y1 12MHz

Commit message: Update BOM
Parts:
- C10, C11, C12, C13, C14, C15, C3, C6, C7, C9: LCSC C307331 -> C1525; MFR. Part # CL05B104KB54PNC -> CL05B104KO5NNNC
- SW1, SW2: LCSC C5117871 -> C498294; MFR. Part # GT-TC060B-H027-L1 -> TS-1064S-A1B2-D4
Changed lines of the file:
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@@
       (effects (font (size 1.27 1.27)) hide)
     )
-    (property "MFR. Part #" "CL05B104KB54PNC " (at 39.37 173.99 0)
-      (effects (font (size 1.27 1.27)) hide)
-    )
-    (property "LCSC" "C307331" (at 39.37 173.99 0)
+    (property "MFR. Part #" "CL05B104KO5NNNC" (at 39.37 173.99 0)
+      (effects (font (size 1.27 1.27)) hide)
+    )
+    (property "LCSC" "C1525" (at 39.37 173.99 0)
       (effects (font (size 1.27 1.27)) hide)
     )
@@
       (effects (font (size 1.27 1.27)) hide)
     )
-    (property "MFR. Part #" "CL05B104KB54PNC " (at 238.76 46.99 0)
-      (effects (font (size 1.27 1.27)) hide)
-    )
-    (property "LCSC" "C307331" (at 238.76 46.99 0)
+    (property "MFR. Part #" "CL05B104KO5NNNC" (at 238.76 46.99 0)
+      (effects (font (size 1.27 1.27)) hide)
+    )
+    (property "LCSC" "C1525" (at 238.76 46.99 0)
       (effects (font (size 1.27 1.27)) hide)
     )
@@
       (effects (font (size 1.27 1.27)) hide)
     )
-    (property "MFR. Part #" "GT-TC060B-H027-L1" (at 245.11 130.81 90)
-      (effects (font (size 1.27 1.27)) hide)
-    )
-    (property "LCSC" "C5117871" (at 245.11 130.81 0)
+    (property "MFR. Part #" "TS-1064S-A1B2-D4" (at 245.11 130.81 90)
+      (effects (font (size 1.27 1.27)) hide)
+    )
+    (property "LCSC" "C498294" (at 245.11 130.81 0)
       (effects (font (size 1.27 1.27)) hide)
     )
@@
       (effects (font (size 1.27 1.27)) hide)
     )
-    (property "MFR. Part #" "CL05B104KB54PNC " (at 62.23 173.99 0)
-      (effects (font (size 1.27 1.27)) hide)
-    )
-    (property "LCSC" "C307331" (at 62.23 173.99 0)
+    (property "MFR. Part #" "CL05B104KO5NNNC" (at 62.23 173.99 0)
+      (effects (font (size 1.27 1.27)) hide)
+    )
+    (property "LCSC" "C1525" (at 62.23 173.99 0)
       (effects (font (size 1.27 1.27)) hide)
     )
@@
       (effects (font (size 1.27 1.27)) hide)
     )
-    (property "MFR. Part #" "GT-TC060B-H027-L1" (at 214.63 130.81 90)
-      (effects (font (size 1.27 1.27)) hide)
-    )
-    (property "LCSC" "C5117871" (at 214.63 130.81 0)
+    (property "MFR. Part #" "TS-1064S-A1B2-D4" (at 214.63 130.81 90)
+      (effects (font (size 1.27 1.27)) hide)
+    )
+    (property "LCSC" "C498294" (at 214.63 130.81 0)
       (effects (font (size 1.27 1.27)) hide)
     )
@@
       )
       (project ""
+        (path "/d5184ecd-32d6-4360-b9b7-27a917b7de38"
+          (reference "C16") (unit 1)
+        )
+      )
+      (project ""
         (path "/d9a18e30-40db-47f3-90f3-96293e98104c"
           (reference "C16") (unit 1)
@@
       (effects (font (size 1.27 1.27)) hide)
     )
-    (property "MFR. Part #" "CL05B104KB54PNC " (at 107.95 173.99 0)
-      (effects (font (size 1.27 1.27)) hide)
-    )
-    (property "LCSC" "C307331" (at 107.95 173.99 0)
+    (property "MFR. Part #" "CL05B104KO5NNNC" (at 107.95 173.99 0)
+      (effects (font (size 1.27 1.27)) hide)
+    )
+    (property "LCSC" "C1525" (at 107.95 173.99 0)
       (effects (font (size 1.27 1.27)) hide)
     )
@@
       (effects (font (size 1.27 1.27)) hide)
     )
-    (property "MFR. Part #" "CL05B104KB54PNC " (at 50.8 151.13 0)
-      (effects (font (size 1.27 1.27)) hide)
-    )
-    (property "LCSC" "C307331" (at 50.8 151.13 0)
+    (property "MFR. Part #" "CL05B104KO5NNNC" (at 50.8 151.13 0)
+      (effects (font (size 1.27 1.27)) hide)
+    )
+    (property "LCSC" "C1525" (at 50.8 151.13 0)
       (effects (font (size 1.27 1.27)) hide)
     )
@@
       (effects (font (size 1.27 1.27)) hide)
     )
-    (property "MFR. Part #" "CL05B104KB54PNC " (at 73.66 173.99 0)
-      (effects (font (size 1.27 1.27)) hide)
-    )
-    (property "LCSC" "C307331" (at 73.66 173.99 0)
+    (property "MFR. Part #" "CL05B104KO5NNNC" (at 73.66 173.99 0)
+      (effects (font (size 1.27 1.27)) hide)
+    )
+    (property "LCSC" "C1525" (at 73.66 173.99 0)
       (effects (font (size 1.27 1.27)) hide)
     )
@@
       (effects (font (size 1.27 1.27)) hide)
     )
-    (property "MFR. Part #" "CL05B104KB54PNC " (at 39.37 151.13 0)
-      (effects (font (size 1.27 1.27)) hide)
-    )
-    (property "LCSC" "C307331" (at 39.37 151.13 0)
+    (property "MFR. Part #" "CL05B104KO5NNNC" (at 39.37 151.13 0)
+      (effects (font (size 1.27 1.27)) hide)
+    )
+    (property "LCSC" "C1525" (at 39.37 151.13 0)
       (effects (font (size 1.27 1.27)) hide)
     )
@@
       (effects (font (size 1.27 1.27)) hide)
     )
-    (property "MFR. Part #" "CL05B104KB54PNC " (at 50.8 173.99 0)
-      (effects (font (size 1.27 1.27)) hide)
-    )
-    (property "LCSC" "C307331" (at 50.8 173.99 0)
+    (property "MFR. Part #" "CL05B104KO5NNNC" (at 50.8 173.99 0)
+      (effects (font (size 1.27 1.27)) hide)
+    )
+    (property "LCSC" "C1525" (at 50.8 173.99 0)
       (effects (font (size 1.27 1.27)) hide)
     )
@@
       (effects (font (size 1.27 1.27)) hide)
     )
-    (property "MFR. Part #" "CL05B104KB54PNC " (at 85.09 173.99 0)
-      (effects (font (size 1.27 1.27)) hide)
-    )
-    (property "LCSC" "C307331" (at 85.09 173.99 0)
+    (property "MFR. Part #" "CL05B104KO5NNNC" (at 85.09 173.99 0)
+      (effects (font (size 1.27 1.27)) hide)
+    )
+    (property "LCSC" "C1525" (at 85.09 173.99 0)
       (effects (font (size 1.27 1.27)) hide)
     )
@@
       (effects (font (size 1.27 1.27)) hide)
     )
-    (property "MFR. Part #" "CL05B104KB54PNC " (at 96.52 173.99 0)
-      (effects (font (size 1.27 1.27)) hide)
-    )
-    (property "LCSC" "C307331" (at 96.52 173.99 0)
+    (property "MFR. Part #" "CL05B104KO5NNNC" (at 96.52 173.99 0)
+      (effects (font (size 1.27 1.27)) hide)
+    )
+    (property "LCSC" "C1525" (at 96.52 173.99 0)
       (effects (font (size 1.27 1.27)) hide)
     )
@@
           (reference "C8") (unit 1)
         )
+      )
+      (project ""
+        (path "/d5184ecd-32d6-4360-b9b7-27a917b7de38"
+          (reference "C8") (unit 1)
+        )
