File: Calcite60/pcb/Calcite60.kicad_pcb (KiCad board)
At the start: 2 copper layers, 226 x 94.2 mm, 191 parts, among them J1 USB_C_Receptacle_USB2.0, J2 Conn_01x02, J3 Conn_01x02, J4 Conn_01x02, J5 Conn_01x02, J6 Conn_01x04, J7 Conn_02x05_Counter_Clockwise, Q1 AO3407, SW1 SW_DPDT_x2, SW2 RESET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

Commit message: Routed
Parts:
- removed the G*** at (45.0, 34.0)
- removed H3: MountingHole, MountingHole:MountingHole_2.2mm_M2
- removed the H5 at (164.1, 105.4)
- added H5: MountingHole, calcite:mouse_bite, F.Cu at (128.9, 86.4)
- added H5: MountingHole, calcite:mouse_bite, F.Cu at (161.4, 86.4)
- added TP1: TestPoint, TestPoint:TestPoint_Pad_D1.5mm, F.Cu at (72.6, 84.4)
- added TP2: TestPoint, TestPoint:TestPoint_Pad_D1.5mm, F.Cu at (72.6, 86.9)
- added TP3: TestPoint, TestPoint:TestPoint_Pad_D1.5mm, F.Cu at (72.6, 89.4)
- added TP4: TestPoint, TestPoint:TestPoint_Pad_D1.5mm, B.Cu at (49.4, 100.7)
- added TP5: TestPoint, TestPoint:TestPoint_Pad_D1.5mm, B.Cu at (49.1, 81.7)
- added TP6: TestPoint, TestPoint:TestPoint_Pad_D1.5mm, B.Cu at (44.9, 100.7)
- added TP7: TestPoint, TestPoint:TestPoint_Pad_D1.5mm, B.Cu at (49.1, 77.2)
- J7: footprint Connector_PinHeader_1.27mm:PinHeader_2x05_P1.27mm_Vertical -> calcite:10pin SWD
- moved G*** 107.0 mm to (232.0, 95.7)
- moved J7 3.85 mm to (125.9, 51.9)
Connections:
- net Battery_sense renamed /MCU/Battery_sense
- J6 pad 1: unconnected-(J6-Pin_1-Pad1) -> VDD
- J7 pad 1: unconnected-(J7-Pin_1-Pad1) -> VDD
- U4 pad 1: State_LED_1 -> COL_3
- U4 pad 10: COL_0 -> COL_1
- U4 pad 12: unconnected-(U4-P0.26-Pad12) -> COL_11
- U4 pad 14: unconnected-(U4-P0.06-Pad14) -> COL_10
- U4 pad 2: State_LED_2 -> COL_4
- U4 pad 20: unconnected-(U4-P0.12-Pad20) -> State_LED_1
- U4 pad 22: unconnected-(U4-P0.07-Pad22) -> State_LED_2
- U4 pad 3: COL_7 -> COL_5
- U4 pad 36: COL_8 -> Net-(U4-P1.00)
- U4 pad 38: COL_9 -> Net-(U4-P1.02)
- U4 pad 40: COL_10 -> Net-(U4-P1.04)
- U4 pad 41: COL_2 -> unconnected-(U4-P0.09/NFC1-Pad41)
- U4 pad 42: COL_11 -> COL_2
- U4 pad 6: COL_5 -> COL_7
- U4 pad 7: COL_4 -> COL_8
- U4 pad 8: COL_3 -> COL_9
- U4 pad 9: COL_1 -> COL_0
Routing:
- net COL_11: track 129.1 -> 337.9 mm, vias 0 -> 1
- net COL_10: track 93.5 -> 277.4 mm, vias 0 -> 2
- net COL_9: track 94.6 -> 260.1 mm, vias 0 -> 3
- net COL_8: track 178.6 -> 312.0 mm, vias 0 -> 3
- net ROW_4: track 227.9 -> 358.1 mm, vias 0 -> 1
- net VDD: track 16.1 -> 130.1 mm, vias 0 -> 1
- net COL_7: track 109.1 -> 221.2 mm, vias 0 -> 3
- net COL_6: track 123.7 -> 220.2 mm, vias 0 -> 3
- net COL_5: track 92.8 -> 166.2 mm, vias 0 -> 3
- net State_LED_1: track 0.00 -> 49.8 mm, vias 0 -> 2
- net COL_4: track 113.5 -> 162.5 mm, vias 1 -> 4
- net State_LED_2: track 0.00 -> 46.0 mm, vias 0 -> 2
- net ROW_3: track 209.0 -> 241.2 mm, vias 0 -> 1
- net COL_3: track 176.2 -> 207.7 mm, vias 0 -> 3
- net COL_0: track 132.2 -> 160.9 mm, vias 0 -> 2
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Other:
- outline, holes or cut-outs redrawn
- board text added: "REV ${REVISION}"
- board text removed: "Rev ${REVISION}"
