File: Calcite60/pcb/Calcite60.kicad_pcb (KiCad board)
At the start: 2 copper layers, 226 x 94.2 mm, 197 parts, among them J1 USB_C_Receptacle_USB2.0, J2 Conn_01x02, J3 Conn_01x02, J4 Conn_01x02, J5 Conn_01x02, J6 Conn_01x04, J7 Conn_02x05_Counter_Clockwise, Q1 AO3407, SW1 SW_DPDT_x2, SW2 RESET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

Commit message: Update BOM
Parts:
- removed the H5 at (128.9, 86.4)
Other:
- board text added: "SideraKB"
- board text removed: "locked"
