File: Calcite60/pcb/Calcite60.kicad_sch (KiCad schematic)
At the start: 26 parts, among them J1 USB_C_Receptacle_USB2.0, U1 RT9013-33GB, U2 SRV05-4

Commit message: Update BOM
Parts:
- H1: renamed from H8; LCSC (none) -> C9900035855; MFR. Part # (none) -> 9774025243R
- H2: renamed from H14; LCSC (none) -> C9900035855; MFR. Part # (none) -> 9774025243R
- H3: renamed from H13; LCSC (none) -> C9900035855; MFR. Part # (none) -> 9774025243R
- H4: renamed from H12; LCSC (none) -> C9900035855; MFR. Part # (none) -> 9774025243R
- H5: renamed from H11; LCSC (none) -> C9900035855; MFR. Part # (none) -> 9774025243R
- H6: renamed from H9; LCSC (none) -> C9900035855; MFR. Part # (none) -> 9774025243R
- H7: renamed from H10; LCSC (none) -> C9900035855; MFR. Part # (none) -> 9774025243R
- U1: LCSC C47773 -> C587158; MFR. Part # RT9013-33GB -> TPRT9013-33GB
- renumbered H3 to H10, H5 to H11, H1 to H12, H2 to H13, H4 to H8, H6 to H9

Commit message: Update Calcite60 Rev2
Parts:
- removed SB1: SolderJumper_2_Open, Jumper:SolderJumper-2_P1.3mm_Open_TrianglePad1.0x1.5mm, symbol Jumper:SolderJumper_2_Open
- added C1: 1uF, Capacitor_SMD:C_0603_1608Metric, symbol Device:C
- added D1: 1N5819, Diode_SMD:D_SOD-323_HandSoldering, symbol Diode:1N5819
- added H14, H15, H16, H17: MountingHole, calcite:MountingWuerth_M2, symbol Mechanical:MountingHole_Pad
- added H18, H19, H20, H21, H22, H23, H24, H25: MountingHole, calcite:mouse_bite, symbol Mechanical:MountingHole
- added J2, J4: Conn_01x02, Connector_PinHeader_2.54mm:PinHeader_1x02_P2.54mm_Vertical, symbol Connector_Generic:Conn_01x02
- added J3, J5: Conn_01x02, Connector_JST:JST_PH_S2B-PH-K_1x02_P2.00mm_Horizontal, symbol Connector_Generic:Conn_01x02
- added J4: Conn_02x05_Counter_Clockwise, Connector_PinHeader_1.27mm:PinHeader_2x05_P1.27mm_Vertical, symbol Connector_Generic:Conn_02x05_Odd_Even
- added J6: Conn_01x04, Connector_PinHeader_2.54mm:PinHeader_1x04_P2.54mm_Vertical, symbol Connector_Generic:Conn_01x04
- added LD1: Blue, LED_SMD:LED_0603_1608Metric, symbol Device:LED
- added Q1: AO3407, Package_TO_SOT_SMD:SOT-23, symbol Transistor_FET:AO3401A
- added R3, R8: 1k, Resistor_SMD:R_0603_1608Metric, symbol Device:R
- added R4: 5.1k, Resistor_SMD:R_0603_1608Metric, symbol Device:R
- added R5: 100k, Resistor_SMD:R_0603_1608Metric, symbol Device:R
- added SW1: SW_DPDT_x2, calcite:9_3.5_3.5 Switch, symbol Switch:SW_DPDT_x2
- added U2: TP4054, Package_TO_SOT_SMD:SOT-23-5, symbol calcite:TP4054
- C2: renamed from C1; footprint Capacitor_SMD:C_0402_1005Metric -> Capacitor_SMD:C_0603_1608Metric
- C3: renamed from C2; footprint Capacitor_SMD:C_0402_1005Metric -> Capacitor_SMD:C_0603_1608Metric
- R1, R2: footprint Resistor_SMD:R_0402_1005Metric -> Resistor_SMD:R_0603_1608Metric
- R6: renamed from R3; footprint Resistor_SMD:R_0402_1005Metric -> Resistor_SMD:R_0603_1608Metric
- renumbered H6 to H10, H7 to H12, H9 to H13, H12 to H3, H3 to H4, H13 to H5, H4 to H6, H10 to H7, H5 to H8, H8 to H9, LD1 to LD2, LD2 to LD3, SB2 to SB1, U2 to U1, U1 to U3
Connections:
- net +5V: now also C1.1, D1.2 (A), LD1.2 (A), Q1.1 (G), R5.1, U2.4 (VCC); no longer C2.1, U3.1 (VIN), U3.3 (EN)
- net GND: now also R6.2, C1.2, J2.2 (Pin_2), J3.2 (Pin_2), J4.2 (Pin_2), J4.3 (Pin_3), J4.5 (Pin_5), J4.9 (Pin_9), J5.2 (Pin_2), J6.4 (Pin_4), R4.2, R5.2, R8.2, U2.2 (GND)
- net at LD2.1 (K), R6.1: no longer LD3.1 (K)
- net +3V3 renamed VDD
- net STATE_LED renamed State_LED_1
- net State_LED_1: no longer LD3.2 (A)
- new net: LD3.1 (K), R8.1
- new net: R4.1, U2.5 (PROG)
- new net: Q1.3 (D), SW1.2 (B)
- new net: C2.1, D1.1 (K), Q1.2 (S), U3.1 (VIN), U3.3 (EN)
- new net: LD1.1 (K), R3.1
- new net: R3.2, U2.1 (~{CHRG})
- new net +BATT: J2.1 (Pin_1), J3.1 (Pin_1), J4.1 (Pin_1), J5.1 (Pin_1), SW1.1 (A), U2.3 (BAT)
- new net SWC: J4.4 (Pin_4), J6.2 (Pin_2)
- new net SWD: J4.2 (Pin_2), J6.3 (Pin_3)
- new net State_LED_2: LD3.2 (A)
- new net ~{RESET}: J4.10 (Pin_10)
- no-connect marks 10 -> 18
Other:
- removed sheet RP2040
- added sheet MCU (mcu.kicad_sch)

Commit message: Routed
Parts:
- removed H3: MountingHole, MountingHole:MountingHole_2.2mm_M2, symbol Mechanical:MountingHole
- added TP1 (x4): TestPoint, TestPoint:TestPoint_Pad_D1.5mm, symbol Connector:TestPoint
- H5: footprint MountingHole:MountingHole_2.2mm_M2 -> calcite:mouse_bite
- J4: footprint Connector_PinHeader_1.27mm:PinHeader_2x05_P1.27mm_Vertical -> calcite:10pin SWD
Connections:
- net +5V: now also TP1.1
- net +BATT: now also TP1.1
- net GND: now also TP1.1
- net VDD: now also J4.1 (Pin_1), J6.1 (Pin_1), TP1.1
