File: Calcite60/pcb/key_matrix.kicad_sch (KiCad schematic)
At the start: 123 parts

Commit message: Update Calcite60 Rev2
Parts:
- added KEY64, KEY65, KEY66: SW_Push_45deg, key-switches:SW_Kailh_Choc_V1_THT_nSilk, symbol Switch:SW_Push_45deg
- KEY1, KEY63: footprint key-switches:SW_Kailh_Choc_V1_THT -> key-switches:SW_Kailh_Choc_V1_THT_nSilk
- KEY10: renamed from KEY50; footprint key-switches:SW_Kailh_Choc_V1_THT -> key-switches:SW_Kailh_Choc_V1_THT_nSilk
- KEY11: renamed from KEY3; footprint key-switches:SW_Kailh_Choc_V1_THT -> key-switches:SW_Kailh_Choc_V1_THT_nSilk
- KEY12: renamed from KEY15; footprint key-switches:SW_Kailh_Choc_V1_THT -> key-switches:SW_Kailh_Choc_V1_THT_nSilk
- KEY13: renamed from KEY27; footprint key-switches:SW_Kailh_Choc_V1_THT -> key-switches:SW_Kailh_Choc_V1_THT_nSilk
- KEY14: renamed from KEY39; footprint key-switches:SW_Kailh_Choc_V1_THT -> key-switches:SW_Kailh_Choc_V1_THT_nSilk
- KEY15: renamed from KEY51; footprint key-switches:SW_Kailh_Choc_V1_THT -> key-switches:SW_Kailh_Choc_V1_THT_nSilk
- KEY16: renamed from KEY4; footprint key-switches:SW_Kailh_Choc_V1_THT -> key-switches:SW_Kailh_Choc_V1_THT_nSilk
- KEY17: renamed from KEY16; footprint key-switches:SW_Kailh_Choc_V1_THT -> key-switches:SW_Kailh_Choc_V1_THT_nSilk
- KEY18: renamed from KEY28; footprint key-switches:SW_Kailh_Choc_V1_THT -> key-switches:SW_Kailh_Choc_V1_THT_nSilk
- KEY19: renamed from KEY40; footprint key-switches:SW_Kailh_Choc_V1_THT -> key-switches:SW_Kailh_Choc_V1_THT_nSilk
- KEY2: renamed from KEY13; footprint key-switches:SW_Kailh_Choc_V1_THT -> key-switches:SW_Kailh_Choc_V1_THT_nSilk
- KEY20: renamed from KEY52; footprint key-switches:SW_Kailh_Choc_V1_THT -> key-switches:SW_Kailh_Choc_V1_THT_nSilk
- KEY21: renamed from KEY53; footprint key-switches:SW_Kailh_Choc_V1_THT -> key-switches:SW_Kailh_Choc_V1_THT_nSilk
- KEY22: renamed from KEY5; footprint key-switches:SW_Kailh_Choc_V1_THT -> key-switches:SW_Kailh_Choc_V1_THT_nSilk
- KEY23: renamed from KEY17; footprint key-switches:SW_Kailh_Choc_V1_THT -> key-switches:SW_Kailh_Choc_V1_THT_nSilk
- KEY24: renamed from KEY29; footprint key-switches:SW_Kailh_Choc_V1_THT -> key-switches:SW_Kailh_Choc_V1_THT_nSilk
- KEY25: renamed from KEY41; footprint key-switches:SW_Kailh_Choc_V1_THT -> key-switches:SW_Kailh_Choc_V1_THT_nSilk
- KEY26: renamed from KEY54; footprint key-switches:SW_Kailh_Choc_V1_THT -> key-switches:SW_Kailh_Choc_V1_THT_nSilk
- KEY27: renamed from KEY6; footprint key-switches:SW_Kailh_Choc_V1_THT -> key-switches:SW_Kailh_Choc_V1_THT_nSilk
- KEY28: renamed from KEY18; footprint key-switches:SW_Kailh_Choc_V1_THT -> key-switches:SW_Kailh_Choc_V1_THT_nSilk
- KEY29: renamed from KEY30; footprint key-switches:SW_Kailh_Choc_V1_THT -> key-switches:SW_Kailh_Choc_V1_THT_nSilk
- KEY3: renamed from KEY25; footprint key-switches:SW_Kailh_Choc_V1_THT -> key-switches:SW_Kailh_Choc_V1_THT_nSilk
- KEY30: renamed from KEY42; footprint key-switches:SW_Kailh_Choc_V1_THT -> key-switches:SW_Kailh_Choc_V1_THT_nSilk
- KEY31: renamed from KEY55; footprint key-switches:SW_Kailh_Choc_V1_THT -> key-switches:SW_Kailh_Choc_V1_THT_nSilk
- KEY32: renamed from KEY56; footprint key-switches:SW_Kailh_Choc_V1_THT -> key-switches:SW_Kailh_Choc_V1_THT_nSilk
- KEY33: renamed from KEY7; footprint key-switches:SW_Kailh_Choc_V1_THT -> key-switches:SW_Kailh_Choc_V1_THT_nSilk
- KEY34: renamed from KEY19; footprint key-switches:SW_Kailh_Choc_V1_THT -> key-switches:SW_Kailh_Choc_V1_THT_nSilk
- KEY35: renamed from KEY31; footprint key-switches:SW_Kailh_Choc_V1_THT -> key-switches:SW_Kailh_Choc_V1_THT_nSilk
- KEY36: renamed from KEY43; footprint key-switches:SW_Kailh_Choc_V1_THT -> key-switches:SW_Kailh_Choc_V1_THT_nSilk
- KEY37: renamed from KEY57; footprint key-switches:SW_Kailh_Choc_V1_THT -> key-switches:SW_Kailh_Choc_V1_THT_nSilk
- KEY38: renamed from KEY58; footprint key-switches:SW_Kailh_Choc_V1_THT -> key-switches:SW_Kailh_Choc_V1_THT_nSilk
- KEY39: renamed from KEY8; footprint key-switches:SW_Kailh_Choc_V1_THT -> key-switches:SW_Kailh_Choc_V1_THT_nSilk
- KEY4: renamed from KEY37; footprint key-switches:SW_Kailh_Choc_V1_THT -> key-switches:SW_Kailh_Choc_V1_THT_nSilk
- KEY40: renamed from KEY20; footprint key-switches:SW_Kailh_Choc_V1_THT -> key-switches:SW_Kailh_Choc_V1_THT_nSilk
- KEY41: renamed from KEY32; footprint key-switches:SW_Kailh_Choc_V1_THT -> key-switches:SW_Kailh_Choc_V1_THT_nSilk
- KEY42: renamed from KEY44; footprint key-switches:SW_Kailh_Choc_V1_THT -> key-switches:SW_Kailh_Choc_V1_THT_nSilk
- KEY43: renamed from KEY59; footprint key-switches:SW_Kailh_Choc_V1_THT -> key-switches:SW_Kailh_Choc_V1_THT_nSilk
- KEY44: renamed from KEY9; footprint key-switches:SW_Kailh_Choc_V1_THT -> key-switches:SW_Kailh_Choc_V1_THT_nSilk
- KEY45: renamed from KEY21; footprint key-switches:SW_Kailh_Choc_V1_THT -> key-switches:SW_Kailh_Choc_V1_THT_nSilk
- KEY46: renamed from KEY33; footprint key-switches:SW_Kailh_Choc_V1_THT -> key-switches:SW_Kailh_Choc_V1_THT_nSilk
- KEY47: renamed from KEY45; footprint key-switches:SW_Kailh_Choc_V1_THT -> key-switches:SW_Kailh_Choc_V1_THT_nSilk
- KEY48: renamed from KEY60; footprint key-switches:SW_Kailh_Choc_V1_THT -> key-switches:SW_Kailh_Choc_V1_THT_nSilk
- KEY49: renamed from KEY10; footprint key-switches:SW_Kailh_Choc_V1_THT -> key-switches:SW_Kailh_Choc_V1_THT_nSilk
- KEY5: renamed from KEY49; footprint key-switches:SW_Kailh_Choc_V1_THT -> key-switches:SW_Kailh_Choc_V1_THT_nSilk
- KEY50: renamed from KEY22; footprint key-switches:SW_Kailh_Choc_V1_THT -> key-switches:SW_Kailh_Choc_V1_THT_nSilk
- KEY51: renamed from KEY34; footprint key-switches:SW_Kailh_Choc_V1_THT -> key-switches:SW_Kailh_Choc_V1_THT_nSilk
- KEY52: renamed from KEY46; footprint key-switches:SW_Kailh_Choc_V1_THT -> key-switches:SW_Kailh_Choc_V1_THT_nSilk
- KEY53: renamed from KEY61; footprint key-switches:SW_Kailh_Choc_V1_THT -> key-switches:SW_Kailh_Choc_V1_THT_nSilk
- KEY54: renamed from KEY11; footprint key-switches:SW_Kailh_Choc_V1_THT -> key-switches:SW_Kailh_Choc_V1_THT_nSilk
- KEY55: renamed from KEY23; footprint key-switches:SW_Kailh_Choc_V1_THT -> key-switches:SW_Kailh_Choc_V1_THT_nSilk
- KEY56: renamed from KEY35; footprint key-switches:SW_Kailh_Choc_V1_THT -> key-switches:SW_Kailh_Choc_V1_THT_nSilk
- KEY57: renamed from KEY47; footprint key-switches:SW_Kailh_Choc_V1_THT -> key-switches:SW_Kailh_Choc_V1_THT_nSilk
- KEY58: renamed from KEY62; footprint key-switches:SW_Kailh_Choc_V1_THT -> key-switches:SW_Kailh_Choc_V1_THT_nSilk
- KEY59: renamed from KEY12; footprint key-switches:SW_Kailh_Choc_V1_THT -> key-switches:SW_Kailh_Choc_V1_THT_nSilk
- KEY6: renamed from KEY2; footprint key-switches:SW_Kailh_Choc_V1_THT -> key-switches:SW_Kailh_Choc_V1_THT_nSilk
- KEY60: renamed from KEY24; footprint key-switches:SW_Kailh_Choc_V1_THT -> key-switches:SW_Kailh_Choc_V1_THT_nSilk
- KEY61: renamed from KEY36; footprint key-switches:SW_Kailh_Choc_V1_THT -> key-switches:SW_Kailh_Choc_V1_THT_nSilk
- KEY62: renamed from KEY48; footprint key-switches:SW_Kailh_Choc_V1_THT -> key-switches:SW_Kailh_Choc_V1_THT_nSilk
- KEY7: renamed from KEY14; footprint key-switches:SW_Kailh_Choc_V1_THT -> key-switches:SW_Kailh_Choc_V1_THT_nSilk
- KEY8: renamed from KEY26; footprint key-switches:SW_Kailh_Choc_V1_THT -> key-switches:SW_Kailh_Choc_V1_THT_nSilk
- KEY9: renamed from KEY38; footprint key-switches:SW_Kailh_Choc_V1_THT -> key-switches:SW_Kailh_Choc_V1_THT_nSilk
- renumbered D38 to D10, D50 to D11, D3 to D12, D15 to D13, D27 to D14, D39 to D15, D51 to D16, D4 to D17, D16 to D18, D28 to D19, D1 to D2, D40 to D20, D52 to D21, D5 to D22, D17 to D23, D29 to D24, D41 to D25, D53 to D26, D6 to D27, D18 to D28, D30 to D29, D13 to D3, D42 to D30, D54 to D31, D7 to D32, D19 to D33, D31 to D34, D43 to D35, D55 to D36, D8 to D37, D20 to D38, D32 to D39, D25 to D4, D44 to D40, D56 to D41, D9 to D42, D21 to D43, D33 to D44, D57 to D46, D10 to D47, D22 to D48, D34 to D49, D37 to D5, D46 to D50, D58 to D51, D11 to D52, D23 to D53, D35 to D54, D47 to D55, D59 to D56, D12 to D57, D24 to D58, D36 to D59, D49 to D6, D48 to D60, D60 to D61, D2 to D7, D14 to D8, D26 to D9
Connections:
- net COL_5: now also KEY26.2, KEY31.1, KEY64.2; no longer KEY26.1, KEY31.2
- net COL_6: now also KEY32.2, KEY37.1, KEY65.2; no longer KEY32.1, KEY37.2
- net COL_7: now also KEY38.2, KEY43.1, KEY66.2; no longer KEY38.1, KEY43.2
- net at D30.2 (A), KEY30.2: now also KEY64.1
- net at D40.2 (A), KEY42.2: now also KEY66.1
- net at D35.2 (A), KEY36.2: now also KEY65.1
- new net: D31.2 (A), KEY26.1, KEY31.2
- new net: D36.2 (A), KEY32.1, KEY37.2
- new net: D41.2 (A), KEY38.1, KEY43.2
Other:
- moved on the sheet: KEY26, KEY30, KEY31, KEY32, KEY36, KEY37, KEY38, KEY42, KEY43
